Commit message: controller_test_0, oscillates, slides

File: src/urdf/robot.urdf (robot description, URDF)
Before this commit: robot robot, 4 links, 3 joints
Joints:
- joint joint_0: limit lower=-1 upper=1 effort=200 velocity=1.0 -> lower=-1 upper=1 effort=1000 velocity=1.0
- joint joint_1: limit lower=-1 upper=1 effort=200 velocity=1.0 -> lower=-1 upper=1 effort=1000 velocity=1.0
- joint joint_2: limit lower=-1.57 upper=1.57 effort=200 velocity=1.0 -> lower=-1.57 upper=1.57 effort=1000 velocity=1.0
